File: attiny-ws8212-plug.kicad_pcb (KiCad board)
At the start: 2 copper layers, 3 parts, among them J1 USB_A, J2 WS2812, U1 ATtiny13-20PU

Commit message: Update
Parts:
- added J3: WS2812, Connector_PinHeader_2.00mm:PinHeader_1x03_P2.00mm_Vertical, F.Cu at (170.1, 122.1)
- added J4: WS2812, Connector_PinHeader_2.00mm:PinHeader_1x03_P2.00mm_Vertical, F.Cu at (180.2, 116.9)
Connections:
- net Net-(J2-Pad2) renamed DataIn
Routing:
- net GND: track 0.00 -> 49.4 mm
- net DataIn: track 0.00 -> 30.4 mm
- added copper zone on B.Cu, net VCC
- added copper zone on F.Cu, net VCC
Other:
- board outline added: 25.4 x 22.9 mm
- board text added: "+"
- board text added: "-"
- board text added: "Copyright (c) 2019 Alejandro Gallo"
- board text added: "In"
